Commit message: feat: Implement EMA joint position action and associated functionalities
- Added EMAJointPositionAction class for joint position control with exponential moving average smoothing.
- Introduced EMAJointPositionActionCfg for configuration settings including smoothing factor.
- Enhanced event handling to track object positions using weak references to avoid delays.
- Added new observation functions for joint position error and tactile proxy fusion.
- Expanded reward functions to include fingertip distance to object, object lifting conditions, and action rate penalties.
- Implemented termination condition for dropped objects based on height and table boundaries.

File: source/humanoid_hand/humanoid_hand/assets/New_URDF_export_description/urdf/New_URDF_export.xacro (robot description, xacro)
@@ -88,5 +88,5 @@
     <origin xyz="-0.0036945196042365014 -0.0016865936108732698 0.0046870721481248045" rpy="0 0 0"/>
     <mass value="0.0019033331833639964"/>
-    <inertia ixx="0.0" iyy="0.0" izz="0.0" ixy="-0.0" iyz="0.0" ixz="0.0"/>
+    <inertia ixx="1e-06" iyy="1e-06" izz="1e-06" ixy="-0.0" iyz="0.0" ixz="0.0"/>
   </inertial>
   <visual>
@@ -108,5 +108,5 @@
     <origin xyz="0.0006578043440388093 0.002756298934102463 0.01152316144300558" rpy="0 0 0"/>
     <mass value="0.0005553551144173429"/>
-    <inertia ixx="0.0" iyy="0.0" izz="0.0" ixy="0.0" iyz="-0.0" ixz="0.0"/>
+    <inertia ixx="1e-06" iyy="1e-06" izz="1e-06" ixy="0.0" iyz="-0.0" ixz="0.0"/>
   </inertial>
   <visual>
@@ -128,5 +128,5 @@
     <origin xyz="-0.0027029859176378873 0.0015940781015286818 0.005832015574820604" rpy="0 0 0"/>
     <mass value="0.002314232689912895"/>
-    <inertia ixx="0.0" iyy="0.0" izz="0.0" ixy="-0.0" iyz="0.0" ixz="0.0"/>
+    <inertia ixx="1e-06" iyy="1e-06" izz="1e-06" ixy="-0.0" iyz="0.0" ixz="0.0"/>
   </inertial>
   <visual>
@@ -168,5 +168,5 @@
     <origin xyz="-0.003330077463916883 -0.002411105311378465 0.00677198635006096" rpy="0 0 0"/>
     <mass value="0.0019033352750190097"/>
-    <inertia ixx="0.0" iyy="0.0" izz="0.0" ixy="0.0" iyz="0.0" ixz="-0.0"/>
+    <inertia ixx="1e-06" iyy="1e-06" izz="1e-06" ixy="0.0" iyz="0.0" ixz="-0.0"/>
   </inertial>
   <visual>
@@ -188,5 +188,5 @@
     <origin xyz="0.0014771000853101325 0.0018048088171991965 0.013173422015586855" rpy="0 0 0"/>
     <mass value="0.0005553551398376143"/>
-    <inertia ixx="0.0" iyy="0.0" izz="0.0" ixy="-0.0" iyz="-0.0" ixz="-0.0"/>
+    <inertia ixx="1e-06" iyy="1e-06" izz="1e-06" ixy="-0.0" iyz="-0.0" ixz="-0.0"/>
   </inertial>
   <visual>
@@ -208,5 +208,5 @@
     <origin xyz="-0.0020740129128638523 0.0008162221421355227 0.007803938698609875" rpy="0 0 0"/>
     <mass value="0.0023142301158833177"/>
-    <inertia ixx="0.0" iyy="0.0" izz="0.0" ixy="-0.0" iyz="0.0" ixz="0.0"/>
+    <inertia ixx="1e-06" iyy="1e-06" izz="1e-06" ixy="-0.0" iyz="0.0" ixz="0.0"/>
   </inertial>
   <visual>
@@ -268,5 +268,5 @@
     <origin xyz="-0.003451516209980696 -0.002233278304004958 0.006772092134296276" rpy="0 0 0"/>
     <mass value="0.0019033302628551495"/>
-    <inertia ixx="0.0" iyy="0.0" izz="0.0" ixy="-0.0" iyz="0.0" ixz="-0.0"/>
+    <inertia ixx="1e-06" iyy="1e-06" izz="1e-06" ixy="-0.0" iyz="0.0" ixz="-0.0"/>
   </inertial>
   <visual>
@@ -288,5 +288,5 @@
     <origin xyz="0.0019193155174742028 0.0017153164675866401 0.013173421980118394" rpy="0 0 0"/>
     <mass value="0.0005553551425762632"/>
-    <inertia ixx="0.0" iyy="0.0" izz="0.0" ixy="-0.0" iyz="-0.0" ixz="-0.0"/>
+    <inertia ixx="1e-06" iyy="1e-06" izz="1e-06" ixy="-0.0" iyz="-0.0" ixz="-0.0"/>
   </inertial>
   <visual>
@@ -308,5 +308,5 @@
     <origin xyz="-0.0019760427506178378 0.002921812974273479 0.007738009794912598" rpy="0 0 0"/>
     <mass value="0.002314230055006617"/>
-    <inertia ixx="0.0" iyy="0.0" izz="0.0" ixy="-0.0" iyz="0.0" ixz="0.0"/>
+    <inertia ixx="1e-06" iyy="1e-06" izz="1e-06" ixy="-0.0" iyz="0.0" ixz="0.0"/>
   </inertial>
   <visual>
@@ -368,5 +368,5 @@
     <origin xyz="-0.0027656231817524343 -0.0011316368308406152 0.005252369213118613" rpy="0 0 0"/>
     <mass value="0.0019033246740478476"/>
-    <inertia ixx="0.0" iyy="0.0" izz="0.0" ixy="-0.0" iyz="0.0" ixz="-0.0"/>
+    <inertia ixx="1e-06" iyy="1e-06" izz="1e-06" ixy="-0.0" iyz="0.0" ixz="-0.0"/>
   </inertial>
   <visual>
@@ -388,5 +388,5 @@
     <origin xyz="0.0031050093271399043 0.0024096864286983315 0.011196454087814722" rpy="0 0 0"/>
     <mass value="0.0005553551392437952"/>
-    <inertia ixx="0.0" iyy="0.0" izz="0.0" ixy="-0.0" iyz="-0.0" ixz="-0.0"/>
+    <inertia ixx="1e-06" iyy="1e-06" izz="1e-06" ixy="-0.0" iyz="-0.0" ixz="-0.0"/>
   </inertial>
   <visual>
@@ -408,5 +408,5 @@
     <origin xyz="-0.0016358581286405743 0.001967218457827354 0.006215753454319822" rpy="0 0 0"/>
     <mass value="0.00231422981504397"/>
-    <inertia ixx="0.0" iyy="0.0" izz="0.0" ixy="0.0" iyz="0.0" ixz="-0.0"/>
+    <inertia ixx="1e-06" iyy="1e-06" izz="1e-06" ixy="0.0" iyz="0.0" ixz="-0.0"/>
   </inertial>
   <visual>
@@ -468,5 +468,5 @@
     <origin xyz="-0.003296225590801106 -0.006582898875138021 0.005592010280368742" rpy="0 0 0"/>
     <mass value="0.002531144718261794"/>
-    <inertia ixx="0.0" iyy="0.0" izz="0.0" ixy="0.0" iyz="0.0" ixz="-0.0"/>
+    <inertia ixx="1e-06" iyy="1e-06" izz="1e-06" ixy="0.0" iyz="0.0" ixz="-0.0"/>
   </inertial>
   <visual>
@@ -488,5 +488,5 @@
     <origin xyz="0.0018930116944578766 -0.014614922867036959 0.0029856270141793064" rpy="0 0 0"/>
     <mass value="0.0007523194454609623"/>
-    <inertia ixx="0.0" iyy="0.0" izz="0.0" ixy="0.0" iyz="0.0" ixz="-0.0"/>
+    <inertia ixx="1e-06" iyy="1e-06" izz="1e-06" ixy="0.0" iyz="0.0" ixz="-0.0"/>
   </inertial>
   <visual>
@@ -508,5 +508,5 @@
     <origin xyz="-0.0019457264466740815 -0.008167025756820878 0.0011558588435874387" rpy="0 0 0"/>
     <mass value="0.0026899841295638023"/>
-    <inertia ixx="0.0" iyy="0.0" izz="0.0" ixy="-0.0" iyz="0.0" ixz="0.0"/>
+    <inertia ixx="1e-06" iyy="1e-06" izz="1e-06" ixy="-0.0" iyz="0.0" ixz="0.0"/>
   </inertial>
   <visual>
